File: ForgeX/HBM_G0V48C15/revA/HBM_G0V48C15 .kicad_pcb (KiCad board)
At the start: 2 copper layers, 32.2 x 69.6 mm, 25 parts, among them J1 Conn_02x05_Odd_Even, J2 Screw_Terminal_01x03, U7 AMS1117-3.3

Commit message: schematic
Parts:
- added C11: 10uF, Capacitor_SMD:C_1206_3216Metric_Pad1.33x1.80mm_HandSolder, F.Cu at (223.3, 65.2)
- added C12: 1uF, Capacitor_SMD:C_1206_3216Metric_Pad1.33x1.80mm_HandSolder, F.Cu at (223.3, 68.6)
- added C13: 0.1u, Capacitor_SMD:C_0603_1608Metric_Pad1.08x0.95mm_HandSolder, F.Cu at (228.4, 71.5)
- added D3: D, Diode_THT:D_DO-35_SOD27_P7.62mm_Horizontal, F.Cu at (221.8, 61.8)
- added D4: SD103AWS_C5345966, EasyEDA:SOD-323_L1.7-W1.3-LS2.5-RD, F.Cu at (228.4, 64.8)
- added D5: SD103AWS_C5345966, EasyEDA:SOD-323_L1.7-W1.3-LS2.5-RD, F.Cu at (228.4, 67.4)
- added Q1: 80N02F, EasyEDA:PDFN-8_L6.0-W5.0-P1.27-BL-A, F.Cu at (224.8, 46.0)
- added Q2: 80N02F, EasyEDA:PDFN-8_L6.0-W5.0-P1.27-BL-A, F.Cu at (214.6, 73.8)
- added R10: 1K, Resistor_SMD:R_1206_3216Metric_Pad1.30x1.75mm_HandSolder, F.Cu at (223.2, 75.2)
- added R2: 10K, Resistor_SMD:R_2512_6332Metric_Pad1.40x3.35mm_HandSolder, F.Cu at (215.7, 62.5)
- added R27: 60k, Resistor_SMD:R_0603_1608Metric_Pad0.98x0.95mm_HandSolder, F.Cu at (228.4, 74.0)
- added R3: 10K, Resistor_SMD:R_2512_6332Metric_Pad1.40x3.35mm_HandSolder, F.Cu at (215.7, 67.4)
- added R9: 1K, Resistor_SMD:R_1206_3216Metric_Pad1.30x1.75mm_HandSolder, F.Cu at (223.2, 71.9)
- added U1: EG2131_C5240691, EasyEDA:SOP-8_L4.9-W3.9-P1.27-LS6.0-BL, F.Cu at (211.7, 46.1)
- added U2: INA199xxDCK, Package_TO_SOT_SMD:SOT-363_SC-70-6, F.Cu at (228.2, 77.1)
- R1: value 5m -> 1m

Commit message: Fabrication ready layout and design
Parts:
- removed C2, C3: 1n, Capacitor_SMD:C_0603_1608Metric_Pad1.08x0.95mm_HandSolder
- removed C20: 10u, Capacitor_SMD:C_2225_5664Metric
- removed D3: D, Diode_THT:D_DO-35_SOD27_P7.62mm_Horizontal
- removed the R27 at (174.7, 86.5)
- removed R28: 150k, Resistor_SMD:R_1206_3216Metric_Pad1.30x1.75mm_HandSolder
- removed U7: AMS1117-3.3, Package_TO_SOT_SMD:SOT-89-3
- added C14: 100n, Capacitor_SMD:C_0603_1608Metric_Pad1.08x0.95mm_HandSolder, B.Cu at (183.9, 80.3)
- added C4: 10u, Capacitor_SMD:C_1210_3225Metric_Pad1.33x2.70mm_HandSolder, B.Cu at (179.9, 69.8)
- added C5: 2.2n, Capacitor_SMD:C_1206_3216Metric_Pad1.33x1.80mm_HandSolder, B.Cu at (166.7, 79.0)
- added C6: 2.2n, Capacitor_SMD:C_1206_3216Metric_Pad1.33x1.80mm_HandSolder, B.Cu at (192.3, 79.0)
- added D6: SS310, Diode_SMD:D_SMA, F.Cu at (165.8, 91.2)
- added H3: MountingHole, MountingHole:MountingHole_2.2mm_M2_DIN965, F.Cu at (193.6, 71.9)
- added H4: MountingHole, MountingHole:MountingHole_2.2mm_M2_DIN965, F.Cu at (166.0, 71.9)
- added R30: 6, Resistor_SMD:R_1206_3216Metric_Pad1.30x1.75mm_HandSolder, B.Cu at (170.5, 80.4)
- added U3: AMS1117-5.0, Package_TO_SOT_SMD:SOT-89-3, F.Cu at (192.8, 105.5)
- C13: value 0.1u -> 4.7n; moved to B.Cu
- C9: value 47n -> 4.7n; moved to B.Cu
- D1, D2: moved to B.Cu
- Q1, Q2: value 80N02F -> NMOS; footprint EasyEDA:PDFN-8_L6.0-W5.0-P1.27-BL-A -> liblocal:DFN5x6; moved to B.Cu
- R1: value 1m -> 10k; footprint Resistor_SMD:R_2512_6332Metric_Pad1.40x3.35mm_HandSolder -> Resistor_SMD:R_0603_1608Metric_Pad0.98x0.95mm_HandSolder
- R10, R9: footprint Resistor_SMD:R_1206_3216Metric_Pad1.30x1.75mm_HandSolder -> Resistor_SMD:R_0603_1608Metric_Pad0.98x0.95mm_HandSolder
- R11, R12: value 10 -> 47; footprint Resistor_SMD:R_1206_3216Metric_Pad1.30x1.75mm_HandSolder -> Resistor_SMD:R_0603_1608Metric_Pad0.98x0.95mm_HandSolder; moved to B.Cu
- R2: value 10K -> 20k; footprint Resistor_SMD:R_2512_6332Metric_Pad1.40x3.35mm_HandSolder -> Resistor_SMD:R_0603_1608Metric_Pad0.98x0.95mm_HandSolder
- R26: value 3.3k -> 2.7k; moved to B.Cu
- R27: value 60k -> 47k; footprint Resistor_SMD:R_0603_1608Metric_Pad0.98x0.95mm_HandSolder -> Resistor_SMD:R_1206_3216Metric_Pad1.30x1.75mm_HandSolder; moved to B.Cu
- R29: value 150k -> 6
- R3: value 10K -> 6; footprint Resistor_SMD:R_2512_6332Metric_Pad1.40x3.35mm_HandSolder -> Resistor_SMD:R_0603_1608Metric_Pad0.98x0.95mm_HandSolder
- U2: value INA199xxDCK -> ACS712xLCTR-20A; footprint Package_TO_SOT_SMD:SOT-363_SC-70-6 -> Package_SO:SOIC-8_3.9x4.9mm_P1.27mm; moved to B.Cu
- moved C11 61.6 mm to (170.5, 97.1), turned to 180 degrees
- moved U1 61.5 mm to (170.5, 91.9)
- moved D4 58.5 mm to (183.6, 102.5), turned to 90 degrees
- moved D5 58.4 mm to (181.8, 102.6), turned to 90 degrees
- moved R3 57.8 mm to (165.8, 96.4), turned to -90 degrees
- moved C12 56.2 mm to (170.0, 86.4), turned to 180 degrees
- moved R27 54.2 mm to (175.6, 86.5)
- moved R9 52.7 mm to (183.6, 106.7), turned to -90 degrees
- moved R10 52.0 mm to (181.8, 106.6), turned to -90 degrees
- moved C13 47.9 mm to (181.9, 83.1)
- moved U2 47.8 mm to (180.4, 78.6), turned to -90 degrees
- moved Q1 47.4 mm to (187.2, 74.8), turned to 180 degrees
- moved R2 47.3 mm to (179.1, 92.3), turned to 90 degrees
- moved Q2 43.1 mm to (171.6, 74.8), turned to 180 degrees
- moved G*** 32.1 mm to (185.2, 96.2)
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Connections:
- C10 pad 1: /Shunt+ -> GNDPWR
- C11 pad 1: /Shunt+ -> GNDPWR
- C12 pad 1: Phase -> Phase+
- C13 pad 1: +3.3V -> Net-(U2-FILTER)
- C38 pad 1: +3.3V -> +5V
- D4 pad 2: /Shunt+ -> GNDPWR
- D5 pad 2: /Shunt+ -> GNDPWR
- J2 pad 2: Phase -> Phase-
- Q1 pad 1: Phase -> Phase+
- Q1 pad 2: Phase -> Net-(D2-A)
- Q1 pad 3: Phase -> GNDPWR
- Q2 pad 1: /Shunt+ -> VDCH
- Q2 pad 2: /Shunt+ -> Net-(D1-A)
- Q2 pad 3: /Shunt+ -> Phase+
- R1 pad 1: /Shunt+ -> Csense
- R1 pad 2: GNDPWR -> Net-(U2-VIOUT)
- R2 pad 1: Net-(U2-REF) -> GND
- R2 pad 2: GND -> Csense
- R27 pad 1: Phase -> Phase+
- R29 pad 2: Phase -> Phase+
- R3 pad 1: +3.3V -> Net-(D6-A)
- R3 pad 2: Net-(U2-REF) -> +12V
- R4 pad 1: Phase -> Phase+
- R5 pad 1: /Shunt+ -> GNDPWR
- R8 pad 1: /Shunt+ -> GNDPWR
- U1 pad 4: /Shunt+ -> GNDPWR
- U1 pad 6: Phase -> Phase+
- U2 pad 1: Net-(U2-REF) -> Phase-
- U2 pad 2: unconnected-(U2-GND-Pad2) -> Phase-
- U2 pad 3: +3.3V -> Phase+
- U2 pad 4: /Shunt+ -> Phase+
- U2 pad 5: GNDPWR -> GND
- U2 pad 6: Csense -> Net-(U2-FILTER)
Routing:
- net /Shunt+: track 95.7 -> 0.00 mm, vias 16 -> 0
- net (no net): track 61.2 -> 0.00 mm, vias 4 -> 0
- net GNDPWR: track 10.8 -> 53.9 mm, vias 28 -> 25
- net +5V: track 0.00 -> 40.9 mm, vias 0 -> 1
- net Phase: track 37.2 -> 0.00 mm, vias 21 -> 0
- net Net-(D4-K): track 0.00 -> 26.8 mm, vias 0 -> 2
- net Net-(D5-K): track 0.00 -> 23.1 mm, vias 0 -> 2
- net +3.3V: track 21.6 -> 0.00 mm
- net VDCH: track 16.5 -> 0.00 mm, vias 25 -> 22
- net Phase+: track 0.00 -> 15.5 mm, vias 0 -> 23
- net Csense: track 35.1 -> 21.7 mm, vias 2 -> 0
- net Net-(U2-VIOUT): track 0.00 -> 9.32 mm, vias 0 -> 1
- net Net-(D6-K): track 0.00 -> 5.62 mm
- net +12V: track 45.5 -> 49.8 mm
- net Phase_Cnd: track 25.3 -> 29.2 mm
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- added copper zone on B.Cu, net Phase+
- added copper zone on F.Cu, net Phase+
- added copper zone on B.Cu, net Phase-
- added copper zone on F.Cu, net Phase-
- removed copper zone on B.Cu, net /Shunt+
- removed copper zone on F.Cu, net /Shunt+
- removed copper zone on B.Cu, net Phase
- removed copper zone on F.Cu, net Phase
