File: ForgeX/HBM_G0V48C15/revA/HBM_G0V48C15 .kicad_sch (KiCad schematic)
At the start: 24 parts, among them J1 Conn_02x05_Odd_Even, J2 Screw_Terminal_01x03, U7 AMS1117-3.3

Commit message: schematic
Parts:
- removed R28, R29: 150k, Resistor_SMD:R_1206_3216Metric_Pad1.30x1.75mm_HandSolder, symbol Device:R
- added C11: 10uF, Capacitor_SMD:C_1206_3216Metric_Pad1.33x1.80mm_HandSolder, symbol Device:C
- added C12: 1uF, Capacitor_SMD:C_1206_3216Metric_Pad1.33x1.80mm_HandSolder, symbol Device:C
- added C13: 0.1u, Capacitor_SMD:C_0603_1608Metric_Pad1.08x0.95mm_HandSolder, symbol Device:C
- added D3: D, Diode_THT:D_DO-35_SOD27_P7.62mm_Horizontal, symbol Device:D
- added D4, D5: SD103AWS_C5345966, EasyEDA:SOD-323_L1.7-W1.3-LS2.5-RD, symbol EasyEDA:SD103AWS_C5345966
- added Q1, Q2: 80N02F, EasyEDA:PDFN-8_L6.0-W5.0-P1.27-BL-A, symbol EasyEDA:80N02F
- added R10, R9: 1K, Resistor_SMD:R_1206_3216Metric_Pad1.30x1.75mm_HandSolder, symbol Device:R
- added R2, R3: 10K, Resistor_SMD:R_2512_6332Metric_Pad1.40x3.35mm_HandSolder, symbol Device:R
- added U1: EG2131_C5240691, EasyEDA:SOP-8_L4.9-W3.9-P1.27-LS6.0-BL, symbol EasyEDA:EG2131_C5240691
- added U2: INA199xxDCK, Package_TO_SOT_SMD:SOT-363_SC-70-6, symbol Amplifier_Current:INA199xxDCK
- R1: value 5m -> 1m
- R27: value 150k -> 60k; footprint Resistor_SMD:R_1206_3216Metric_Pad1.30x1.75mm_HandSolder -> Resistor_SMD:R_0603_1608Metric_Pad0.98x0.95mm_HandSolder
Connections:
- net +12V: now also C11.2, D3.2 (A), U1.1 (VCC)
- net +3.3V: now also C13.1, R3.1, U2.3 (V+)
- net Csense: now also U2.6
- net GND: now also C13.2, R2.2
- net GNDPWR: now also U2.5 (-)
- net HIN: now also R9.2
- net HS_GateSig: now also U1.7 (HO)
- net LIN: now also R10.2
- net LS_GateSig: now also U1.5 (LO)
- net Phase: now also R27.1, C12.1, Q1.1 (S), Q1.2 (S), Q1.3 (S), Q2.5 (D), Q2.6 (D), Q2.7 (D), Q2.8 (D), U1.6 (VS)
- net Phase_Cnd: now also R27.2; no longer R27.1
- net Shunt+: now also C11.1, D4.2 (A), D5.2 (A), Q2.1 (S), Q2.2 (S), Q2.3 (S), U1.4 (GND), U2.4 (+)
- net VDCH: now also Q1.5 (D), Q1.6 (D), Q1.7 (D), Q1.8 (D)
- net at C3.1, D1.2 (A), R11.2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: now also Q1.4 (G)
- net at C2.1, D2.2 (A), R12.2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: now also Q2.4 (G)
- new net: D4.1 (K), R9.1, U1.2 (HIN)
- new net: C12.2, D3.1 (K), U1.8 (VB)
- new net: R2.1, R3.2, U2.1 (REF)
- new net: D5.1 (K), R10.1, U1.3 (~{LIN})
Other:
- moved on the sheet: C37, C38, U7

Commit message: Fabrication ready layout and design
Parts:
- removed C2, C3: 1n, Capacitor_SMD:C_0603_1608Metric_Pad1.08x0.95mm_HandSolder, symbol Device:C
- removed C20: 10u, Capacitor_SMD:C_2225_5664Metric, symbol Device:C
- removed D3: D, Diode_THT:D_DO-35_SOD27_P7.62mm_Horizontal, symbol Device:D
- removed Q1, Q2: 80N02F, EasyEDA:PDFN-8_L6.0-W5.0-P1.27-BL-A, symbol EasyEDA:80N02F
- removed U2: INA199xxDCK, Package_TO_SOT_SMD:SOT-363_SC-70-6, symbol Amplifier_Current:INA199xxDCK
- removed U7: AMS1117-3.3, Package_TO_SOT_SMD:SOT-89-3, symbol Regulator_Linear:AMS1117-3.3
- added C14: 100n, Capacitor_SMD:C_0603_1608Metric_Pad1.08x0.95mm_HandSolder, symbol Device:C
- added C4: 10u, Capacitor_SMD:C_1210_3225Metric_Pad1.33x2.70mm_HandSolder, symbol Device:C
- added C5, C6: 2.2n, Capacitor_SMD:C_1206_3216Metric_Pad1.33x1.80mm_HandSolder, symbol Device:C
- added D6: SS310, Diode_SMD:D_SMA, symbol Device:D_Schottky
- added H3, H4: MountingHole, MountingHole:MountingHole_2.2mm_M2_DIN965, symbol Mechanical:MountingHole
- added Q1, Q2: NMOS, liblocal:DFN5x6, symbol Simulation_SPICE:NMOS
- added R29, R30: 6, Resistor_SMD:R_1206_3216Metric_Pad1.30x1.75mm_HandSolder, symbol Device:R
- added U2: ACS712xLCTR-20A, Package_SO:SOIC-8_3.9x4.9mm_P1.27mm, symbol Sensor_Current:ACS712xLCTR-20A
- added U3: AMS1117-5.0, Package_TO_SOT_SMD:SOT-89-3, symbol Regulator_Linear:AMS1117-5.0
- C13: value 0.1u -> 4.7n
- C9: value 47n -> 4.7n
- R1: value 1m -> 10k; footprint Resistor_SMD:R_2512_6332Metric_Pad1.40x3.35mm_HandSolder -> Resistor_SMD:R_0603_1608Metric_Pad0.98x0.95mm_HandSolder
- R10, R9: footprint Resistor_SMD:R_1206_3216Metric_Pad1.30x1.75mm_HandSolder -> Resistor_SMD:R_0603_1608Metric_Pad0.98x0.95mm_HandSolder
- R11, R12: value 10 -> 47; footprint Resistor_SMD:R_1206_3216Metric_Pad1.30x1.75mm_HandSolder -> Resistor_SMD:R_0603_1608Metric_Pad0.98x0.95mm_HandSolder
- R2: value 10K -> 20k; footprint Resistor_SMD:R_2512_6332Metric_Pad1.40x3.35mm_HandSolder -> Resistor_SMD:R_0603_1608Metric_Pad0.98x0.95mm_HandSolder
- R26: value 3.3k -> 2.7k
- R27: value 60k -> 47k; footprint Resistor_SMD:R_0603_1608Metric_Pad0.98x0.95mm_HandSolder -> Resistor_SMD:R_1206_3216Metric_Pad1.30x1.75mm_HandSolder
- R3: value 10K -> 6; footprint Resistor_SMD:R_2512_6332Metric_Pad1.40x3.35mm_HandSolder -> Resistor_SMD:R_0603_1608Metric_Pad0.98x0.95mm_HandSolder
Connections:
- net +12V: now also R3.2, U3.3 (VI)
- net Csense: now also R1.1, R2.2
- net GND: now also R2.1, C14.2, U2.5 (GND), U3.1 (GND); no longer R2.2
- net GNDPWR: now also C10.1, C11.1, D4.2 (A), D5.2 (A), R5.1, R8.1, U1.4 (GND), C4.2, C6.1, Q1.3 (S); no longer R1.2
- net VDCH: now also C4.1, C5.1, Q2.1 (D)
- net at C12.2, U1.8 (VB): now also D6.1 (K)
- net at D1.2 (A), R11.2, R4.2: now also Q2.2 (G)
- net at D2.2 (A), R12.2, R5.2: now also Q1.2 (G)
- removed net +3.3V: C13.1, C38.1, R3.1
- net Phase renamed Phase+
- net Phase+: now also Q1.1 (D), Q2.3 (S), R29.2, R30.2, U2.3 (IP-), U2.4 (IP-); no longer J2.2 (Pin_2)
- removed net Shunt+: C10.1, C11.1, D4.2 (A), D5.2 (A), R1.1, R5.1, R8.1, U1.4 (GND)
- new net: C5.2, R30.1
- new net: D6.2 (A), R3.1
- new net: C13.1, U2.6 (FILTER)
- new net: R1.2, U2.7 (VIOUT)
- new net: C6.2, R29.1
- new net +5V: C14.1, C38.1, U2.8 (VCC), U3.2 (VO)
- new net Phase-: J2.2 (Pin_2), U2.1 (IP+), U2.2 (IP+)
Other:
- moved on the sheet: C9, D1, D2, R11, R12, R27, R4, R5
